File: Analog Synth/AR - Attack Release.sch (EAGLE design)
At the start: 44 parts, among them IC1 78L05Z, IC2 TL084P, T1 2N3904, T2 2N3904, T3 2N3904, T4 2N3904, T5 2N3904

Commit message: added Attack-Release schematic with a JFET-based VCA that won't work. I will need to modify the schematic for a bual board.
Parts:
- removed T2, T3, T4, T5: 2N3904, transistor:2N3904
- removed U$5, U$6: 2N7000, !synth_sch:2N7000
- added IC4: TL084P, linear:TL084P
- added OFFSET-IN, V-CTRL, V-IN, V-OUT: I/O, !synth_sch:MONO_JACK
- added Q1: 2N5485, transistor-fet:2N5485
- added R18, R19, R25: 100k, resistor:R-US_0204/7
- added R20, R23: 1k, resistor:R-US_0204/7
- added R21: 220k, resistor:R-US_0204/7
- added R22: 100k, pot:TRIM_US-B64Y
- added R24: 10k, resistor:R-US_0204/7
- added R26: 68.8k, resistor:R-US_0204/7
- added U$1, U$2: 2N7000, !synth_sch:2N7000
- C1: value 0.1µ -> 1µ; device capacitor-wima:C2.5/2 -> rcl:C-US025-050X050
- C8: value 10µ -> 33µ
- C9: value 1m -> 1000u
- R11: value 47k -> 10k; device resistor:R-US_0204/7 -> pot:TRIM_US-B64Y
- R12: device pot:TRIM_US-B64Y -> resistor:R-US_0204/7
Connections:
- removed net N$22: IC2D.OUT, R16.2, R17.1
- new net N$24: IC4C.OUT, R16.1, R19.2
- new net N$27: Q1.G, R19.1
- new net N$28: IC2D.+IN, OFFSET-IN.P2
- new net N$29: R20.2, V-OUT.P2
- new net N$30: R22.A, R23.2
- new net N$31: IC4B.+IN, V-IN.P2
- new net N$32: IC4B.-IN, IC4B.OUT, Q1.D, R26.2
- new net N$33: IC4A.+IN, V-CTRL.P2
- new net N$34: IC4D.+IN, Q1.S, R24.2
- new net N$35: IC4C.+IN, R21.2, R25.2, R26.1
- new net N$36: IC4D.-IN, IC4D.OUT, R20.1
- net +12V: no longer T2.C, T3.C, T4.C, T5.C
- net -12V: now also R21.1
- net GND: now also OFFSET-IN.P$1, OFFSET-IN.P3, R11.E, R18.1, R23.1, R24.1, U$1.S, U$2.S, V-CTRL.P$1, V-CTRL.P3, V-IN.P$1, V-IN.P3, V-OUT.P$1; no longer IC2D.+IN, R8.1, U$5.S, U$6.S
- net N$13: now also IC2D.-IN, IC2D.OUT, R12.1; no longer T2.E, T3.B
- net N$14: now also IC4A.OUT, R22.S, R25.1; no longer T4.E, T5.B
- net N$16: now also IC4C.-IN, R16.2, R18.2; no longer IC2B.+IN, R8.2, T5.E
- net N$17: now also R11.S; no longer IC2B.-IN, IC2B.OUT
- net N$19: now also R8.1; no longer R11.1
- net N$20: now also R12.2, R14.2, R15.1, R8.2; no longer R11.2, R12.A
- net N$23: now also R17.1; no longer R12.E, R12.S
- net N$3: now also U$1.G, U$2.G; no longer U$5.G, U$6.G
- net N$4: now also U$1.D; no longer U$5.D
- net N$5: now also IC4A.-IN, R22.E; no longer IC2D.-IN, R14.2, R15.1, R16.1
- net N$6: now also IC2B.-IN, IC2B.OUT, R11.A; no longer T3.E, T4.B
- net N$7: now also U$2.D; no longer U$6.D
- net N$8: now also IC2B.+IN; no longer T2.B
