File: Analog Synth/Front Panels/VCO-v1.brd (EAGLE design)
At the start: 10 parts

Commit message: split up VCO-v1 over multiple pages. cleaning things up.
Parts:
- added E$10: (no value), !synth_panel:KNOB_BOSS_MEDIUM
- added E$12, E$29, E$30, E$31, E$33: (no value), !synth_panel:3.5MM_JACK_TAYDA
- added E$13: (no value), !synth_panel:KNBO_BOSS_SMALL
- added E$14: (no value), !synth_panel:POTENTIOMETER_TAYDA_6MM
- added E$15, E$17, E$20, E$23, E$25, E$27, E$37, E$38, E$39, E$40: (no value), !synth_panel:LED_3MM
- E$6: device !synth_panel:4U_1 -> !synth_panel:4U_2
- E$8: device !synth_panel:3.5MM_JACK_TAYDA -> !synth_panel:KNOB_BOSS-LARGE
- moved E$9 114.3 mm to (36.8, 143.5)
- moved E$7 84.8 mm to (36.8, 97.8)
- moved E$11 70.3 mm to (36.8, 128.3)
- moved E$3 60.2 mm to (20.3, 63.5)
- moved E$2 59.7 mm to (14.0, 92.7)
- moved E$1 31.6 mm to (43.2, 64.8), turned to 0 degrees
- moved E$5 27.9 mm to (36.8, 113.0)
- moved E$8 24.4 mm to (27.9, 27.9), turned to 180 degrees
- moved E$4 24.2 mm to (36.8, 82.5)
Routing:
- net S$3: track 0.00 -> 78.9 mm
- net S$2: track 0.00 -> 78.5 mm
- net S$1: track 0.00 -> 66.3 mm
Other:
- board text added: "CV-A MANUAL"
- board text added: "CV-B ATTN"
- board text added: "LFO"
- board text added: "PWM"
- board text added: "PWM-OFFSET"
- board text added: "RST"
- board text added: "Ramp Down"
- board text added: "Ramp Up"
- board text added: "VCO"
- board text removed: "CV-A Coarse"
- board text removed: "CV-A Fine"
- board text removed: "Ramp"
