File: Analog Synth/Front Panels/Dual Sequencer.brd (EAGLE design)
At the start: 245 x 150 mm, 24 parts

Commit message: I realized that I have more work to do on the schematic than I do have to do on the Panel. The circuit needs to be figured out exactly first. But that shouldn't take long. The filter may pose a slight challenge. Also I kind of want a mid-range VCO for both channels
Parts:
- added E$25, E$26, E$27, E$28, E$29, E$30, E$31, E$32: (no value), !synth_panel:POTENTIOMETER_TAYDA_6MM
Changed lines of the file:
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@@
 <wire x1="200" y1="149" x2="200" y2="1" width="0.4064" layer="19"/>
 <wire x1="231" y1="149" x2="231" y2="1" width="0.4064" layer="19"/>
+<dimension x1="14" y1="93" x2="14" y2="112" x3="-7" y3="102.5" textsize="1.778" layer="19"/>
 </plain>
 <attributes>
@@
 <element name="E$23" library="!synth_panel" package="LED_3MM" value="" x="200" y="58"/>
 <element name="E$24" library="!synth_panel" package="LED_3MM" value="" x="231" y="58"/>
+<element name="E$25" library="!synth_panel" package="POTENTIOMETER_TAYDA_6MM" value="" x="14" y="75" rot="R90"/>
+<element name="E$26" library="!synth_panel" package="POTENTIOMETER_TAYDA_6MM" value="" x="45" y="75" rot="R90"/>
+<element name="E$27" library="!synth_panel" package="POTENTIOMETER_TAYDA_6MM" value="" x="76" y="75" rot="R90"/>
+<element name="E$28" library="!synth_panel" package="POTENTIOMETER_TAYDA_6MM" value="" x="107" y="75" rot="R90"/>
+<element name="E$29" library="!synth_panel" package="POTENTIOMETER_TAYDA_6MM" value="" x="231" y="75" rot="R270"/>
+<element name="E$30" library="!synth_panel" package="POTENTIOMETER_TAYDA_6MM" value="" x="200" y="75" rot="R270"/>
+<element name="E$31" library="!synth_panel" package="POTENTIOMETER_TAYDA_6MM" value="" x="169" y="75" rot="R270"/>
+<element name="E$32" library="!synth_panel" package="POTENTIOMETER_TAYDA_6MM" value="" x="138" y="75" rot="R270"/>
 </elements>
 <signals>
