File: Analog Synth/Front Panels/VCO-v2.brd (EAGLE design)
At the start: 25 parts

Commit message: VCO-v2
Parts:
- E$11: value (none) -> PWM-MAN
Other:
- board text added: "PWM-MAN"
- board text removed: "CV-A-ATTN"
Changed lines of the file:
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@@
 <board>
 <plain>
-<text x="8.89" y="165.1" size="2.54" layer="104">CV-A</text>
-<text x="8.89" y="149.86" size="2.54" layer="104">CV-B</text>
-<text x="8.89" y="134.62" size="2.54" layer="104">CV-C</text>
-<text x="8.89" y="119.38" size="2.54" layer="104">CV-PWM</text>
-<text x="8.89" y="74.93" size="2.54" layer="104">TRIANGLE</text>
-<text x="8.89" y="59.69" size="2.54" layer="104">PWM</text>
-<text x="8.89" y="90.17" size="2.54" layer="104">SINE</text>
-<text x="27.94" y="167.64" size="2.54" layer="104">CV-A-ATTN</text>
-<text x="27.94" y="138.43" size="2.54" layer="104">CV-B-ATTN</text>
-<text x="27.94" y="109.22" size="2.54" layer="104">CV-C-ATTN</text>
-<text x="24.13" y="80.01" size="2.54" layer="104">CV-PWM-ATTN</text>
+<text x="10.16" y="165.1" size="2.54" layer="104">CV-A</text>
+<text x="10.16" y="149.86" size="2.54" layer="104">CV-B</text>
+<text x="10.16" y="134.62" size="2.54" layer="104">CV-C</text>
+<text x="5.08" y="119.38" size="2.54" layer="104">CV-PWM</text>
+<text x="2.54" y="74.93" size="2.54" layer="104">TRIANGLE</text>
+<text x="12.7" y="59.69" size="2.54" layer="104">PWM</text>
+<text x="11.43" y="90.17" size="2.54" layer="104">SINE</text>
+<text x="29.21" y="80.01" size="2.54" layer="104">PWM-MAN</text>
+<text x="27.94" y="167.64" size="2.54" layer="104">CV-B-ATTN</text>
+<text x="27.94" y="138.43" size="2.54" layer="104">CV-C-ATTN</text>
+<text x="24.13" y="109.22" size="2.54" layer="104">CV-PWM-ATTN</text>
 <text x="21.59" y="43.18" size="2.54" layer="104">CV-A-MANUAL</text>
 </plain>
@@
 <element name="E$8" library="!synth_panel" package="KNBO_BOSS_SMALL" value="" x="38.1" y="97.79"/>
 <element name="E$9" library="!synth_panel" package="KNBO_BOSS_SMALL" value="" x="38.1" y="127"/>
-<element name="E$11" library="!synth_panel" package="KNBO_BOSS_SMALL" value="" x="38.1" y="156.21"/>
+<element name="E$11" library="!synth_panel" package="KNBO_BOSS_SMALL" value="PWM-MAN" x="38.1" y="156.21"/>
 </elements>
 <signals>

Commit message: VCO-v2 added switch for range
Parts:
- added E$12: (no value), !synth_panel:TOGGLE_SWITCH_TAYDA
Changed lines of the file:
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@@
 <element name="E$9" library="!synth_panel" package="KNBO_BOSS_SMALL" value="" x="38.1" y="127"/>
 <element name="E$11" library="!synth_panel" package="KNBO_BOSS_SMALL" value="PWM-MAN" x="38.1" y="156.21"/>
+<element name="E$12" library="!synth_panel" package="TOGGLE_SWITCH_TAYDA" value="" x="11.43" y="100.33" rot="R90"/>
 </elements>
 <signals>
