File: Analog Synth/Front Panels/CBS - Cigar Box Sequencer - 8 step.brd (EAGLE design)
At the start: 65 parts

Commit message: CBS: chem and front panel of the cigar box
Parts:
- added E$49, E$67, E$68, E$69, E$70, E$71, E$72, E$73: (no value), !synth_panel:TOGGLE_SWITCH_TAYDA
Changed lines of the file:
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@@
 <text x="115" y="125" size="2.54" layer="104">CLK</text>
 <text x="21" y="136" size="2.54" layer="104">INT-OSC</text>
+<wire x1="2" y1="52.5" x2="243" y2="52.5" width="0.4064" layer="20"/>
 </plain>
 <attributes>
@@
 <element name="E$17" library="!synth_panel" package="TOGGLE_SWITCH_TAYDA" value="" x="45" y="141" rot="R90"/>
 <element name="E$47" library="!synth_panel" package="LED_3MM" value="" x="28" y="133"/>
+<element name="E$49" library="!synth_panel" package="TOGGLE_SWITCH_TAYDA" value="" x="14" y="52.5" rot="R180"/>
+<element name="E$67" library="!synth_panel" package="TOGGLE_SWITCH_TAYDA" value="" x="45" y="52.5" rot="R180"/>
+<element name="E$68" library="!synth_panel" package="TOGGLE_SWITCH_TAYDA" value="" x="76" y="52.5" rot="R180"/>
+<element name="E$69" library="!synth_panel" package="TOGGLE_SWITCH_TAYDA" value="" x="107" y="52.5" rot="R180"/>
+<element name="E$70" library="!synth_panel" package="TOGGLE_SWITCH_TAYDA" value="" x="138" y="52.5" rot="R180"/>
+<element name="E$71" library="!synth_panel" package="TOGGLE_SWITCH_TAYDA" value="" x="169" y="52.5" rot="R180"/>
+<element name="E$72" library="!synth_panel" package="TOGGLE_SWITCH_TAYDA" value="" x="200" y="52.5" rot="R180"/>
+<element name="E$73" library="!synth_panel" package="TOGGLE_SWITCH_TAYDA" value="" x="231" y="52.5" rot="R180"/>
 </elements>
 <signals>
