File: Senior Design/circuit.sch (EAGLE design)
At the start: 24 parts, among them IC1 74HC164N, IC2 ATMEGA328P, IC3 ATTINY24A, Q1 16 MHz

Commit message: working on senior design PCB
Parts:
- removed JP3: (no value), pinhead:PINHD-2X3
- added C1, C2: 20pf, rcl:C-EU025-024X044
Connections:
- net +5V: now also JP2.1, JP2.3; no longer JP3.1, JP3.3
- net GND: now also C1.1, C2.1, JP2.5, JP2.7; no longer JP3.5, JP3.6
- net N$1: now also JP2.4; no longer JP3.4
- net N$2: now also JP2.2; no longer JP3.2
- net N$5: now also C1.2
- net N$6: now also C2.2
Other:
- moved on the sheet: IC1, IC2, JP2, Q1, R1, R10, R11, R12, R13, R14, R15, R16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

Commit message: working on senior design circuit and pcb
Parts:
- removed IC1: 74HC164N, 74xx-us:74HC164N
- removed R10, R11, R4, R5, R6, R7, R8, R9: 10 kΩ, resistor:R-US_0204/7
- removed R12, R13, R14, R15, R16, R17: 4.7 kΩ, resistor:R-US_0204/7
- added C3, C4, C5, C7: 10nf, rcl:C-EU025-024X044
- added C6: 100uF, rcl:C-US025-050X050
- added JP1: (no value), pinhead:PINHD-1X2/90
- Q1: value 16 MHz -> 16MHz
- R3: value 4.7 kΩ -> 10 kΩ
Connections:
- removed net N$10: R11.1, R2.1, R3.1
- removed net N$11: R14.1, R15.1, R7.1
- removed net N$12: R15.2, R16.1, R8.1
- removed net N$13: R16.2, R17.1, R9.1
- removed net N$14: R12.2, R13.1, R5.1
- removed net N$15: R12.1, R3.2, R4.1
- removed net N$17: R10.1, R17.2
- removed net N$19: IC1A.QF, R8.2
- removed net N$25: IC1A.QB, R4.2
- removed net N$26: IC1A.QC, R5.2
- removed net N$27: IC1A.QD, R6.2
- removed net N$28: IC1A.QE, R7.2
- removed net N$30: IC1A.QG, R9.2
- removed net N$31: IC1A.QH, R10.2
- net +5V: now also C5.2, C6.1, C7.2, JP2.5, JP2.6; no longer IC1A.B, IC1A.CLR, JP2.1, JP2.3
- net GND: now also C3.1, C4.1, C5.1, C6.2, C7.1, JP1.1, JP2.8; no longer JP2.5, R11.2, S1.P
- net N$1: now also IC3.P$2, JP2.3; no longer IC3.P$3
- net N$2: now also IC3.P$3, JP2.1; no longer IC3.P$2
- net N$3: now also IC3.P$10, JP1.2; no longer IC1A.CLK, IC3.P$12
- net N$4: now also IC3.P$5, R2.2; no longer IC1A.A, IC3.P$11
- net N$7: now also C3.2, R2.1, R3.2; no longer R13.2, R14.2, R6.1
- net N$8: no longer S1.S
- net N$9: now also C4.2, IC2.ANALOG_0, R3.1; no longer IC1A.QA, R2.2
Other:
- note removed: "line_out"
- moved on the sheet: IC3, JP2, R2, R3

Commit message: worked on the schematic
Parts:
- removed C7: 10nf, rcl:C-EU025-024X044
- added JP3: (no value), pinhead:PINHD-2X3
Connections:
- net N$1 renamed P_BSI_DATA
- net N$2 renamed P_SWEEP
- removed net N$9: C4.2, IC2.ANALOG_0, R3.1
- new net DATA-READY: IC2.DIGITAL_6(PWM), IC3.P$6
- new net LINE-POSITION: C4.2, IC2.ANALOG_1, R3.1
- new net MISO: IC3.P$8, JP3.1
- new net MOSI: IC3.P$7, JP3.4
- new net P_MOTOR: IC2.DIGITAL_7, JP2.11, JP2.12
- new net P_STEER: IC2.DIGITAL_8, JP2.10, JP2.9
- new net RST: IC3.P$4, JP3.5
- new net SCK: IC3.P$9, JP3.3
- net +5V: now also JP3.2; no longer C7.2
- net GND: now also JP3.6; no longer C7.1
Other:
- note removed: "p_data"
- note removed: "p_sweep"
- moved on the sheet: C1, C2, C3, C4, C5, C6, IC2, JP1, Q1, R1, R2, R3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

Commit message: working on senior design and analog switch
Parts:
- added C7: 4.7uF, rcl:C-US025-050X050
- added C8: 10nf, rcl:C-EU025-024X044
- added C9: 1.1uF, rcl:C-US025-050X050
- added IC1: LM2907, ic-package:DIL14
- added R4: 10 kΩ, resistor:R-US_0204/2V
- added R5: 2.2 kΩ, resistor:R-US_0204/2V
- added R6: 200 kΩ, resistor:R-US_0204/2V
- added R7: 220 kΩ, resistor:R-US_0204/2V
- JP1: device pinhead:PINHD-1X2/90 -> pinhead:PINHD-1X2
- R1, R2, R3: device resistor:R-US_0204/7 -> resistor:R-US_0204/2V
Connections:
- new net FIN: C7.1, JP2.12, R5.2
- new net N$1: C9.1, IC1.3, IC1.4, R6.1
- new net N$12: C8.2, IC1.2
- new net N$9: C7.2, IC1.1, R4.1
- new net V_FREQ: IC1.10, IC1.5, IC2.ANALOG_0, R7.2
- net +5V: now also IC1.8, IC1.9
- net GND: now also C8.1, C9.2, IC1.11, IC1.12, R4.2, R5.1, R6.2, R7.1
- net P_MOTOR: no longer JP2.12
- net P_STEER: no longer JP2.10
Other:
- moved on the sheet: C3, C4, C5, C6, R2, R3
