File: Analog Synth/Echo Chamber/Echo Chamber.brd (EAGLE design)
At the start: 160 x 100 mm, 59 parts, among them IC7 78L05, IC8 TL082P, Q1 2N3906, Q2 2N3906

Commit message: fixed little bug with the Echo Chamber schematic
Parts:
- C22: value 10 µF -> 47 µF
- C23: value 10 µF -> 100 µF
Changed lines of the file:
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@@
 <element name="C6" library="capacitor-wima" package="C5B2.5" value="0.1 µF" x="-57.15" y="-220.98"/>
 <element name="R5" library="resistor" package="0204/7" value="2.7 kΩ" x="-57.15" y="-227.33"/>
-<element name="C22" library="rcl" package="C025-060X050" value="10 µF" x="-58.42" y="-233.68"/>
-<element name="C23" library="rcl" package="C025-060X050" value="10 µF" x="-58.42" y="-242.57"/>
+<element name="C22" library="rcl" package="C025-060X050" value="47 µF" x="-58.42" y="-233.68"/>
+<element name="C23" library="rcl" package="C025-060X050" value="100 µF" x="-58.42" y="-242.57"/>
 <element name="C24" library="capacitor-wima" package="C5B2.5" value="0.1 µF" x="-57.15" y="-248.92"/>
 <element name="LED-AUDIO_IN" library="led" package="LED3MM" value="" x="-59.69" y="-255.27"/>
