File: Strobeoscope/Stroboscope.sch (EAGLE design)
At the start: 279 parts, among them Q2 IRLZ44Z

Commit message: stroboscope
Parts:
- added C1: 10u, rcl:C-US025-050X050
- added C2: 1n, rcl:C-EU025-024X044
- IC1: value (none) -> lm317t
- Q2: value IRLZ44Z -> irf630b
- T1, T2: value (none) -> 2n3904
Connections:
- net GND: now also C1.2, C2.2
- net N$26: now also C2.1
- net N$52: now also C1.1
Other:
- note added: "C1 helps stabalize the LM317T. This is only important when the GATE input is switching the LEDs ON and OFF at moderate frequencies (audio range)."
- note added: "Current Source = (V REF / R1 ) + I ADJ = 1.25 V / R (from datasheet) For R = 1.25 Ohms, Current = 1 Amp. R = R55 R55 should be able to dissipate 1 Watt of power (minimum)"
- note added: "I was having issues with high-freq oscillation in the T1, T2, Q2 input stage. I put C2 in the circuit to reduce the gain at higher frequencies. This seemed to fix the oscillation problem."
- note added: "Supply voltage must be greater than the sum of the following three voltages: + The voltage drop across the MOSFET + The voltage drop of th eLM317T + The voltage drop of the LED network Supply must be able to source 1 A continuously."
- note removed: "Current Source = (V REF / R1 ) + I ADJ = 1.25 V / R1 (from datasheet) For R1 = 1.25 Ohms, Current = 1 Amp."
- moved on the sheet: D1
Changed lines of the file:
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@@
 </classes>
 <parts>
-<part name="IC1" library="v-reg" deviceset="LM317TL" device=""/>
-<part name="Q2" library="transistor-power" deviceset="IRLZ44Z" device=""/>
+<part name="IC1" library="v-reg" deviceset="LM317TL" device="" value="lm317t"/>
+<part name="Q2" library="transistor-power" deviceset="IRLZ44Z" device="" value="irf630b"/>
 <part name="LED1" library="led" deviceset="LED" device="5MM"/>
 <part name="LED2" library="led" deviceset="LED" device="5MM"/>
@@
 <part name="R53" library="rcl" deviceset="R-US_" device="0204/7" value="7.5"/>
 <part name="R54" library="rcl" deviceset="R-US_" device="0204/7" value="7.5"/>
-<part name="SUPPLY1" library="supply2" deviceset="+18V" device=""/>
+<part name="SUPPLY1" library="supply1" deviceset="+24V" device=""/>
 <part name="R55" library="rcl" deviceset="R-US_" device="0411/12" value="1.25"/>
 <part name="SUPPLY2" library="supply2" deviceset="GND" device=""/>
-<part name="T1" library="transistor" deviceset="*-NPN-" device="TO92"/>
-<part name="T2" library="transistor" deviceset="*-NPN-" device="TO92"/>
+<part name="T1" library="transistor" deviceset="*-NPN-" device="TO92" value="2n3904"/>
+<part name="T2" library="transistor" deviceset="*-NPN-" device="TO92" value="2n3904"/>
 <part name="D1" library="diode" deviceset="1N4004" device=""/>
 <part name="SUPPLY3" library="supply2" deviceset="GND" device=""/>
@@
 <part name="R58" library="rcl" deviceset="R-US_" device="0204/7" value="10k"/>
 <part name="SUPPLY5" library="supply2" deviceset="GND" device=""/>
+<part name="C1" library="rcl" deviceset="C-US" device="025-050X050" value="10u"/>
+<part name="C2" library="rcl" deviceset="C-EU" device="025-024X044" value="1n"/>
+<part name="SUPPLY6" library="supply2" deviceset="GND" device=""/>
 </parts>
 <sheets>
 <sheet>
 <plain>
-<text x="85.09" y="162.56" size="1.778" layer="98">Current Source = (V REF / R1 ) + I ADJ = 1.25 V / R1
+<text x="90.17" y="149.86" size="1.778" layer="98">Current Source = (V REF / R1 ) + I ADJ = 1.25 V / R
 (from datasheet)
-For R1 = 1.25 Ohms, Current = 1 Amp.</text>
+For R = 1.25 Ohms, Current = 1 Amp.
+R = R55
+R55 should be able to dissipate 1 Watt of power (minimum)</text>
+<text x="5.08" y="-7.62" size="1.778" layer="98">I was having issues with high-freq oscillation in the T1, T2, Q2 input stage.
+I put C2 in the circuit to reduce the gain at higher frequencies.
+This seemed to fix the oscillation problem.</text>
+<text x="-20.32" y="109.22" size="1.778" layer="98">C1 helps stabalize the LM317T.
+This is only important when the GATE input is switching
+the LEDs ON and OFF at moderate frequencies (audio range).</text>
+<text x="-12.7" y="154.94" size="1.778" layer="98">Supply voltage must be greater than
+the sum of the following three voltages:
++ The voltage drop across the MOSFET
++ The voltage drop of th eLM317T
++ The voltage drop of the LED network
+Supply must be able to source 1 A continuously.</text>
 </plain>
 <instances>
-<instance part="IC1" gate="A" x="64.77" y="165.1"/>
+<instance part="IC1" gate="A" x="64.77" y="165.1" smashed="yes">
+<attribute name="NAME" x="59.69" y="171.45" size="1.778" layer="95"/>
+<attribute name="VALUE" x="59.69" y="168.91" size="1.778" layer="96"/>
+</instance>
 <instance part="Q2" gate="G$1" x="76.2" y="33.02" smashed="yes">
-<attribute name="NAME" x="82.55" y="34.29" size="1.778" layer="95"/>
-<attribute name="VALUE" x="82.55" y="31.75" size="1.778" layer="96"/>
+<attribute name="NAME" x="83.82" y="34.29" size="1.778" layer="95"/>
+<attribute name="VALUE" x="83.82" y="31.75" size="1.778" layer="96"/>
 </instance>
 <instance part="LED1" gate="G$1" x="58.42" y="116.84"/>
@@
 <instance part="R53" gate="G$1" x="571.5" y="73.66" rot="R90"/>
 <instance part="R54" gate="G$1" x="579.12" y="73.66" rot="R90"/>
-<instance part="SUPPLY1" gate="+18V" x="53.34" y="170.18"/>
+<instance part="SUPPLY1" gate="1" x="53.34" y="170.18"/>
 <instance part="R55" gate="G$1" x="78.74" y="157.48" rot="R90"/>
 <instance part="SUPPLY2" gate="GND" x="78.74" y="10.16"/>
 <instance part="T1" gate="G$1" x="27.94" y="30.48" smashed="yes">
-<attribute name="NAME" x="30.48" y="30.48" size="1.778" layer="95"/>
-<attribute name="VALUE" x="17.78" y="35.56" size="1.778" layer="96"/>
+<attribute name="NAME" x="33.02" y="30.48" size="1.778" layer="95"/>
+<attribute name="VALUE" x="33.02" y="27.94" size="1.778" layer="96"/>
 </instance>
 <instance part="T2" gate="G$1" x="45.72" y="30.48" smashed="yes">
-<attribute name="NAME" x="48.26" y="30.48" size="1.778" layer="95"/>
-<attribute name="VALUE" x="35.56" y="35.56" size="1.778" layer="96"/>
+<attribute name="NAME" x="50.8" y="30.48" size="1.778" layer="95"/>
+<attribute name="VALUE" x="50.8" y="27.94" size="1.778" layer="96"/>
 </instance>
-<instance part="D1" gate="1" x="17.78" y="20.32" rot="R90"/>
+<instance part="D1" gate="1" x="12.7" y="20.32" rot="R90"/>
 <instance part="SUPPLY3" gate="GND" x="48.26" y="10.16"/>
 <instance part="R56" gate="G$1" x="30.48" y="45.72" rot="R90"/>
@@
 <instance part="R58" gate="G$1" x="2.54" y="30.48"/>
 <instance part="SUPPLY5" gate="GND" x="0" y="10.16"/>
+<instance part="C1" gate="G$1" x="38.1" y="132.08"/>
+<instance part="C2" gate="G$1" x="20.32" y="22.86"/>
+<instance part="SUPPLY6" gate="GND" x="38.1" y="124.46"/>
 </instances>
 <busses>
@@
 <net name="N$52" class="0">
 <segment>
-<wire x1="139.7" y1="121.92" x2="139.7" y2="137.16" width="0.1524" layer="91"/>
 <pinref part="LED49" gate="G$1" pin="A"/>
 <wire x1="180.34" y1="119.38" x2="180.34" y2="121.92" width="0.1524" layer="91"/>
@@
 <junction x="246.38" y="121.92"/>
 <junction x="259.08" y="121.92"/>
-<wire x1="259.08" y1="121.92" x2="259.08" y2="137.16" width="0.1524" layer="91"/>
 <wire x1="259.08" y1="137.16" x2="200.66" y2="137.16" width="0.1524" layer="91"/>
 <wire x1="200.66" y1="137.16" x2="198.12" y2="137.16" width="0.1524" layer="91"/>
@@
 <junction x="368.3" y="121.92"/>
 <junction x="381" y="121.92"/>
-<wire x1="381" y1="121.92" x2="381" y2="137.16" width="0.1524" layer="91"/>
 <wire x1="381" y1="137.16" x2="320.04" y2="137.16" width="0.1524" layer="91"/>
 <junction x="320.04" y="137.16"/>
@@
 <junction x="487.68" y="121.92"/>
 <junction x="500.38" y="121.92"/>
-<wire x1="500.38" y1="121.92" x2="500.38" y2="137.16" width="0.1524" layer="91"/>
 <wire x1="500.38" y1="137.16" x2="441.96" y2="137.16" width="0.1524" layer="91"/>
 <junction x="441.96" y="137.16"/>
@@
 <junction x="78.74" y="149.86"/>
 <junction x="139.7" y="137.16"/>
+<pinref part="C1" gate="G$1" pin="1"/>
+<wire x1="38.1" y1="134.62" x2="38.1" y2="137.16" width="0.1524" layer="91"/>
+<wire x1="38.1" y1="137.16" x2="78.74" y2="137.16" width="0.1524" layer="91"/>
 </segment>
 </net>
@@
 <segment>
 <pinref part="IC1" gate="A" pin="IN"/>
-<pinref part="SUPPLY1" gate="+18V" pin="+18V"/>
+<pinref part="SUPPLY1" gate="1" pin="+24V"/>
 <wire x1="53.34" y1="167.64" x2="53.34" y2="165.1" width="0.1524" layer="91"/>
 <wire x1="53.34" y1="165.1" x2="57.15" y2="165.1" width="0.1524" layer="91"/>
@@
 <wire x1="0" y1="12.7" x2="0" y2="15.24" width="0.1524" layer="91"/>
 <pinref part="D1" gate="1" pin="A"/>
-<wire x1="17.78" y1="15.24" x2="17.78" y2="17.78" width="0.1524" layer="91"/>
+<wire x1="12.7" y1="15.24" x2="12.7" y2="17.78" width="0.1524" layer="91"/>
 <pinref part="T2" gate="G$1" pin="E"/>
 <wire x1="48.26" y1="25.4" x2="48.26" y2="15.24" width="0.1524" layer="91"/>
 <wire x1="48.26" y1="15.24" x2="30.48" y2="15.24" width="0.1524" layer="91"/>
 <pinref part="T1" gate="G$1" pin="E"/>
-<wire x1="30.48" y1="15.24" x2="17.78" y2="15.24" width="0.1524" layer="91"/>
+<wire x1="30.48" y1="15.24" x2="20.32" y2="15.24" width="0.1524" layer="91"/>
+<wire x1="20.32" y1="15.24" x2="12.7" y2="15.24" width="0.1524" layer="91"/>
 <wire x1="30.48" y1="25.4" x2="30.48" y2="15.24" width="0.1524" layer="91"/>
 <junction x="30.48" y="15.24"/>
@@
 <wire x1="48.26" y1="15.24" x2="78.74" y2="15.24" width="0.1524" layer="91"/>
 <junction x="78.74" y="15.24"/>
-<wire x1="0" y1="15.24" x2="17.78" y2="15.24" width="0.1524" layer="91"/>
-<junction x="17.78" y="15.24"/>
+<wire x1="0" y1="15.24" x2="12.7" y2="15.24" width="0.1524" layer="91"/>
+<junction x="12.7" y="15.24"/>
 <wire x1="0" y1="15.24" x2="-7.62" y2="15.24" width="0.1524" layer="91"/>
 <junction x="0" y="15.24"/>
+<pinref part="C2" gate="G$1" pin="2"/>
+<wire x1="20.32" y1="17.78" x2="20.32" y2="15.24" width="0.1524" layer="91"/>
+<junction x="20.32" y="15.24"/>
+</segment>
+<segment>
+<pinref part="C1" gate="G$1" pin="2"/>
+<pinref part="SUPPLY6" gate="GND" pin="GND"/>
 </segment>
 </net>
@@
 <segment>
 <pinref part="T1" gate="G$1" pin="B"/>
-<wire x1="25.4" y1="30.48" x2="17.78" y2="30.48" width="0.1524" layer="91"/>
+<wire x1="25.4" y1="30.48" x2="20.32" y2="30.48" width="0.1524" layer="91"/>
 <pinref part="D1" gate="1" pin="C"/>
-<wire x1="17.78" y1="30.48" x2="7.62" y2="30.48" width="0.1524" layer="91"/>
-<wire x1="17.78" y1="22.86" x2="17.78" y2="30.48" width="0.1524" layer="91"/>
-<junction x="17.78" y="30.48"/>
+<wire x1="20.32" y1="30.48" x2="12.7" y2="30.48" width="0.1524" layer="91"/>
+<wire x1="12.7" y1="30.48" x2="7.62" y2="30.48" width="0.1524" layer="91"/>
+<wire x1="12.7" y1="22.86" x2="12.7" y2="30.48" width="0.1524" layer="91"/>
+<junction x="12.7" y="30.48"/>
 <pinref part="R58" gate="G$1" pin="2"/>
-</segment>
-</net>
+<pinref part="C2" gate="G$1" pin="1"/>
+<wire x1="20.32" y1="25.4" x2="20.32" y2="30.48" width="0.1524" layer="91"/>
+<junction x="20.32" y="30.48"/>
+</segment>
+</net>

Commit message: stroboscope
Connections:
- new net +24V: R56.2, R57.2
- net +18V: no longer R56.2, R57.2
Changed lines of the file:
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@@
 <part name="R56" library="rcl" deviceset="R-US_" device="0204/7" value="2.2k"/>
 <part name="R57" library="rcl" deviceset="R-US_" device="0204/7" value="2.2k"/>
-<part name="SUPPLY4" library="supply2" deviceset="+18V" device=""/>
 <part name="R58" library="rcl" deviceset="R-US_" device="0204/7" value="10k"/>
 <part name="SUPPLY5" library="supply2" deviceset="GND" device=""/>
@@
 <part name="C2" library="rcl" deviceset="C-EU" device="025-024X044" value="1n"/>
 <part name="SUPPLY6" library="supply2" deviceset="GND" device=""/>
+<part name="SUPPLY7" library="supply1" deviceset="+24V" device=""/>
 </parts>
 <sheets>
@@
 <instance part="R56" gate="G$1" x="30.48" y="45.72" rot="R90"/>
 <instance part="R57" gate="G$1" x="48.26" y="45.72" rot="R90"/>
-<instance part="SUPPLY4" gate="+18V" x="30.48" y="63.5"/>
 <instance part="R58" gate="G$1" x="2.54" y="30.48"/>
 <instance part="SUPPLY5" gate="GND" x="0" y="10.16"/>
@@
 <instance part="C2" gate="G$1" x="20.32" y="22.86"/>
 <instance part="SUPPLY6" gate="GND" x="38.1" y="124.46"/>
+<instance part="SUPPLY7" gate="1" x="30.48" y="63.5"/>
 </instances>
 <busses>
@@
 <wire x1="53.34" y1="165.1" x2="57.15" y2="165.1" width="0.1524" layer="91"/>
 </segment>
-<segment>
-<pinref part="R56" gate="G$1" pin="2"/>
-<wire x1="30.48" y1="50.8" x2="30.48" y2="58.42" width="0.1524" layer="91"/>
-<pinref part="R57" gate="G$1" pin="2"/>
-<wire x1="48.26" y1="50.8" x2="48.26" y2="58.42" width="0.1524" layer="91"/>
-<wire x1="48.26" y1="58.42" x2="30.48" y2="58.42" width="0.1524" layer="91"/>
-<pinref part="SUPPLY4" gate="+18V" pin="+18V"/>
-<wire x1="30.48" y1="58.42" x2="30.48" y2="60.96" width="0.1524" layer="91"/>
-<junction x="30.48" y="58.42"/>
-</segment>
 </net>
 <net name="N$235" class="0">
@@
 </segment>
 </net>
+<net name="+24V" class="0">
+<segment>
+<pinref part="R56" gate="G$1" pin="2"/>
+<wire x1="30.48" y1="50.8" x2="30.48" y2="58.42" width="0.1524" layer="91"/>
+<pinref part="R57" gate="G$1" pin="2"/>
+<wire x1="48.26" y1="50.8" x2="48.26" y2="58.42" width="0.1524" layer="91"/>
+<wire x1="48.26" y1="58.42" x2="30.48" y2="58.42" width="0.1524" layer="91"/>
+<wire x1="30.48" y1="58.42" x2="30.48" y2="60.96" width="0.1524" layer="91"/>
+<junction x="30.48" y="58.42"/>
+<pinref part="SUPPLY7" gate="1" pin="+24V"/>
+</segment>
+</net>
