File: Analog Synth/VCA-v2/VCA-v2a.brd (EAGLE design)
At the start: 50 x 50 mm, 43 parts, among them IC2 TL084D, T1 DMMT3904W, T2 MMBT2222ALT1

Commit message: final gerbers
Parts:
- moved R24 2.25 mm to (18.5, 9.75), turned to 45 degrees
- moved R23 1.59 mm to (34.3, 29.2)
Routing:
- net N$22: track 4.72 -> 2.67 mm
- net N$24: track 44.0 -> 45.5 mm
- net N$30: track 4.70 -> 5.61 mm
Other:
- board text added: "2016 June"
- board text added: "Ryan Jensen"
- board text added: "VCA-v2"
Changed lines of the file:
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@@
 <rectangle x1="0" y1="0" x2="7.3025" y2="49.8475" layer="30"/>
 <rectangle x1="40.005" y1="0" x2="49.8475" y2="49.8475" layer="30"/>
+<wire x1="0" y1="0" x2="0" y2="50" width="0" layer="20"/>
+<text x="39.0525" y="30.7975" size="3.81" layer="26" font="vector" rot="MR0">VCA-v2</text>
+<text x="37.1475" y="12.3825" size="1.778" layer="26" font="vector" rot="SMR270" align="center">Ryan Jensen</text>
+<text x="9.2075" y="9.8425" size="1.778" layer="26" font="vector" rot="SMR270" align="center">2016 June</text>
 </plain>
 <attributes>
@@
 <attribute name="VALUE" x="34.9885" y="27.813" size="0.6096" layer="27"/>
 </element>
-<element name="R23" library="resistor" package="R0603" value="100k" x="34.29" y="30.7975" smashed="yes" rot="R90">
-<attribute name="NAME" x="35.306" y="31.6865" size="0.6096" layer="25"/>
-<attribute name="VALUE" x="35.306" y="30.988" size="0.6096" layer="27"/>
+<element name="R23" library="resistor" package="R0603" value="100k" x="34.29" y="29.21" smashed="yes" rot="R90">
+<attribute name="NAME" x="35.306" y="30.099" size="0.6096" layer="25"/>
+<attribute name="VALUE" x="35.306" y="29.4005" size="0.6096" layer="27"/>
 </element>
 <element name="AUDIO-OUT" library="!synth_sch" package="MONO_JACK" value="I/O" x="15.24" y="12.7" smashed="yes">
@@
 <attribute name="NAME" x="11.4935" y="10.4775" size="0.6096" layer="25" ratio="10" rot="R270"/>
 </element>
-<element name="R24" library="resistor" package="R0603" value="3.3k" x="20.6375" y="10.4775" smashed="yes">
-<attribute name="NAME" x="22.2885" y="10.7315" size="0.6096" layer="25"/>
-<attribute name="VALUE" x="22.2885" y="10.033" size="0.6096" layer="27"/>
+<element name="R24" library="resistor" package="R0603" value="3.3k" x="18.507990625" y="9.74950625" smashed="yes" rot="R45">
+<attribute name="NAME" x="20.13081875" y="8.87404375" size="0.6096" layer="25" rot="R45"/>
+<attribute name="VALUE" x="21.259734375" y="9.015128125" size="0.6096" layer="27" rot="R45"/>
 </element>
 <element name="T1" library="!synth_sch" package="SOT363" value="DMMT3904W" x="32.0675" y="24.765" smashed="yes" rot="R270">
@@
 <via x="43.18" y="5.08" extent="1-16" drill="0.8128"/>
 <via x="40.64" y="2.54" extent="1-16" drill="0.8128"/>
-<wire x1="43.18" y1="15.24" x2="40.64" y2="17.78" width="0" layer="19" extent="1-1"/>
-<wire x1="40.64" y1="12.7" x2="43.18" y2="15.24" width="0" layer="19" extent="1-1"/>
-<wire x1="43.18" y1="10.16" x2="40.64" y2="12.7" width="0" layer="19" extent="1-1"/>
-<wire x1="40.64" y1="7.62" x2="43.18" y2="10.16" width="0" layer="19" extent="1-1"/>
-<wire x1="43.18" y1="5.08" x2="40.64" y2="7.62" width="0" layer="19" extent="1-1"/>
-<wire x1="40.64" y1="2.54" x2="43.18" y2="5.08" width="0" layer="19" extent="1-1"/>
-<wire x1="43.18" y1="20.32" x2="40.64" y2="17.78" width="0" layer="19" extent="1-1"/>
 </signal>
 <signal name="+12V">
@@
 <wire x1="32.385" y1="27.94" x2="32.385" y2="28.36" width="0.3048" layer="1"/>
 <wire x1="32.385" y1="28.36" x2="32.805" y2="27.94" width="0.4064" layer="1"/>
-<wire x1="32.805" y1="27.94" x2="34.29" y2="27.94" width="0.4064" layer="1"/>
-<via x="34.29" y="27.94" extent="1-16" drill="0.6096" diameter="0.6096"/>
-<wire x1="34.29" y1="27.94" x2="30.48" y2="31.75" width="0.4064" layer="16"/>
+<via x="34.925" y="26.67" extent="1-16" drill="0.6096" diameter="0.6096"/>
+<wire x1="34.925" y1="26.67" x2="30.48" y2="31.75" width="0.4064" layer="16"/>
 <wire x1="30.48" y1="31.75" x2="27.94" y2="31.75" width="0.4064" layer="16"/>
 <wire x1="27.94" y1="31.75" x2="26.67" y2="33.02" width="0.4064" layer="16"/>
@@
 <via x="33.235" y="45.72" extent="1-16" drill="0.6096"/>
 <wire x1="33.235" y1="45.72" x2="30.695" y2="45.72" width="0.4064" layer="1"/>
+<wire x1="34.925" y1="26.67" x2="33.655" y2="26.67" width="0.4064" layer="1"/>
+<wire x1="33.655" y1="26.67" x2="33.655" y2="26.3525" width="0.4064" layer="1"/>
 </signal>
 <signal name="N$26">
@@
 <wire x1="31.115" y1="31.4325" x2="31.115" y2="32.325" width="0.4064" layer="1"/>
 <wire x1="32.385" y1="30.06" x2="32.59" y2="30.06" width="0.4064" layer="1"/>
-<wire x1="32.59" y1="30.06" x2="34.29" y2="29.9475" width="0.4064" layer="1"/>
+<wire x1="34.29" y1="28.36" x2="34.085" y2="28.36" width="0.4064" layer="1"/>
+<wire x1="34.085" y1="28.36" x2="32.385" y2="30.06" width="0.4064" layer="1"/>
 </signal>
 <signal name="N$31">
@@
 <contactref element="IC2" pad="7"/>
 <contactref element="R24" pad="2"/>
-<wire x1="21.4875" y1="10.4775" x2="21.4875" y2="12.7" width="0.4064" layer="1"/>
-<via x="34.29" y="33.3375" extent="1-16" drill="0.6096" diameter="0.6096"/>
+<wire x1="19.10903125" y1="10.350546875" x2="21.4875" y2="12.7" width="0.4064" layer="1"/>
+<via x="34.29" y="32.0675" extent="1-16" drill="0.6096" diameter="0.6096"/>
 <wire x1="36.195" y1="24.765" x2="24.765" y2="24.765" width="0.4064" layer="16"/>
 <wire x1="24.765" y1="24.765" x2="24.13" y2="24.13" width="0.4064" layer="16"/>
@@
 <wire x1="21.59" y1="14.9225" x2="21.4875" y2="14.82" width="0.4064" layer="1"/>
 <wire x1="21.4875" y1="14.82" x2="21.4875" y2="12.7" width="0.4064" layer="1"/>
-<wire x1="32.385" y1="32.325" x2="32.6425" y2="32.0675" width="0.4064" layer="1"/>
-<wire x1="36.195" y1="32.7025" x2="36.195" y2="24.765" width="0.4064" layer="16"/>
-<wire x1="34.29" y1="31.6475" x2="33.6125" y2="32.325" width="0.4064" layer="1"/>
-<wire x1="33.6125" y1="32.325" x2="32.385" y2="32.325" width="0.4064" layer="1"/>
-<wire x1="34.29" y1="31.6475" x2="34.29" y2="33.3375" width="0.4064" layer="1"/>
-<wire x1="36.195" y1="32.7025" x2="35.56" y2="33.3375" width="0.4064" layer="16"/>
-<wire x1="35.56" y1="33.3375" x2="34.29" y2="33.3375" width="0.4064" layer="16"/>
+<wire x1="36.195" y1="31.4325" x2="36.195" y2="24.765" width="0.4064" layer="16"/>
+<wire x1="34.29" y1="30.06" x2="34.29" y2="32.0675" width="0.4064" layer="1"/>
+<wire x1="36.195" y1="31.4325" x2="35.56" y2="32.0675" width="0.4064" layer="16"/>
+<wire x1="35.56" y1="32.0675" x2="34.29" y2="32.0675" width="0.4064" layer="16"/>
+<wire x1="34.29" y1="32.0675" x2="32.6425" y2="32.0675" width="0.4064" layer="1"/>
+<wire x1="32.6425" y1="32.0675" x2="32.385" y2="32.325" width="0.4064" layer="1"/>
 </signal>
 <signal name="N$32">
@@
 <contactref element="R24" pad="1"/>
 <contactref element="LED-AUDIO-OUT" pad="A"/>
-<wire x1="19.7875" y1="10.4775" x2="15.24" y2="9.2075" width="0.4064" layer="1"/>
+<wire x1="17.906946875" y1="9.1484625" x2="15.24" y2="9.2075" width="0.4064" layer="1"/>
 </signal>
 </signals>
