File: Analog Synth/VCA-v2/VCA-v2.1.brd (EAGLE design)
At the start: 50 x 50 mm, 43 parts, among them IC2 TL084D, T1 DMMT3904W, T2 MMBT2222ALT1

Commit message: ScreamFilter v1.0; TODO: Add LEDs to ScreamFilter...   updated VCA-v2 for some reason.
Parts:
- T2: value MMBT2222ALT1 -> DSC2001
Changed lines of the file:
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@@
 <attribute name="VALUE" x="33.825" y="23.97" size="0.6096" layer="27"/>
 </element>
-<element name="T2" library="transistor" package="SOT23-BEC" value="MMBT2222ALT1" x="17.78" y="43.815" smashed="yes" rot="R270">
+<element name="T2" library="transistor" package="SOT23-BEC" value="DSC2001" x="17.78" y="43.815" smashed="yes" rot="R270">
 <attribute name="NAME" x="15.875" y="44.1325" size="0.6096" layer="25" rot="R180"/>
 <attribute name="VALUE" x="15.875" y="44.7675" size="0.6096" layer="27" rot="R180"/>
