File: XPhone/Input_Board/Input Board.sch (KiCad schematic (older format))
At the start: 26 parts

Commit message: working on XPhone/Input_Board
Parts:
- removed C? (x3): 10n, symbol C_Small
- added C1, C10, C12, C14, C16, C17, C19, C2, C20, C21, C22, C23, C24, C25, C26, C4, C5, C6, C8, C9: 10n, Capacitors_SMD:C_0603, symbol C_Small
- added C18: 10µ, Capacitors_Tantalum_SMD:CP_Tantalum_Case-B_EIA-3528-21_Wave, symbol CP1
- added J10, J4, J9: ENV, Pin_Headers:Pin_Header_Straight_1x01_Pitch2.54mm, symbol CONN_01X01
- added J11, J12, J6: PULSE, Pin_Headers:Pin_Header_Straight_1x01_Pitch2.54mm, symbol CONN_01X01
- added J2, J7, J8: AUDIO, Pin_Headers:Pin_Header_Straight_1x01_Pitch2.54mm, symbol CONN_01X01
- added L2, L3, L4: Input Coil, Pin_Headers:Pin_Header_Straight_1x02_Pitch2.54mm, symbol L
- added Q2, Q4, Q5, Q6, Q7, Q8: BC847CW, TO_SOT_Packages_SMD:SOT-323_SC-70_Handsoldering, symbol MMBT3904
- added R12, R22, R23, R26, R28, R6: 10M, Resistors_SMD:R_0603, symbol R
- added R13, R24, R25, R27, R29, R9: 1M, Resistors_SMD:R_0603, symbol R
- added R15, R17, R30, R31, R32, R33: 100k, Resistors_SMD:R_0603, symbol R
- added R18, R19, R2: 4.7, Resistors_SMD:R_0603, symbol R
- added R20, R21, R4: 10k, Resistors_SMD:R_0603, symbol R
- added R7: 0, Resistors_SMD:R_0603, symbol R
- added RV2, RV3, RV4: 10k, Potentiometers:Potentiometer_Trimmer_Bourns_3296W, symbol POT
- added unit 2 of U1
- added U2: 78L05, TO_SOT_Packages_THT:TO-92_Inline_Narrow_Oval, symbol 78L05
- added unit 3 of U3
- added unit 2 of U3
- added unit 4 of U3
- added unit 3 of U4
- added unit 2 of U4
- added unit 4 of U4
- added unit 5 of U4
- added unit 6 of U4
- added U5: LM833, Housings_DIP:DIP-8_W7.62mm, symbol LM358
- C11, C13, C15, C3, C7: renamed from C?; footprint (none) -> Capacitors_SMD:C_0603
- J1, J3, J5: renamed from J?; footprint (none) -> Pin_Headers:Pin_Header_Straight_1x01_Pitch2.54mm
- L1: renamed from L?; footprint (none) -> Pin_Headers:Pin_Header_Straight_1x02_Pitch2.54mm
- Q1, Q3: renamed from Q?; footprint TO_SOT_Packages_SMD:SOT-23 -> TO_SOT_Packages_SMD:SOT-323_SC-70_Handsoldering
- R1, R10, R11, R14, R16, R3, R5, R8: renamed from R?; footprint (none) -> Resistors_SMD:R_0603
- RV1: renamed from RV?; footprint (none) -> Potentiometers:Potentiometer_Trimmer_Bourns_3296W
- U1: renamed from U?; footprint (none) -> Housings_DIP:DIP-8_W7.62mm
- U3, U4: renamed from U?; footprint (none) -> Housings_DIP:DIP-14_W7.62mm
Connections:
- net +12V: now also C1.1, C1.2, C10.1, C10.2, C12.2, C2.1, C2.2, C5.1, C5.2, C6.1, C6.2, C9.1, C9.2, R15.1, R30.1, R31.1, U1.4 (V-), U1.8 (V+), U2.1 (VI), U3.11 (V-), U3.11 (V-), U3.11 (V-), U3.4 (V+), U3.4 (V+), U3.4 (V+), U5.4 (V-), U5.4 (V-), U5.8 (V+), U5.8 (V+); no longer C11.2
- net GND: now also C11.2, C12.1, C17.2, C18.2, R7.2, U2.2 (GND), U4.7 (GND), U4.7 (GND), U4.7 (GND), U4.7 (GND), U4.7 (GND)
- net GNDA: now also C14.2, C19.2, C20.2, C23.2, C24.2, C4.2, L2.1, L3.1, L4.1, Q4.2 (E), Q7.2 (E), Q8.2 (E), R13.2, R18.2, R19.2, R2.2, R27.2, R29.2, R7.1
- net VCC: now also C17.1, C18.1, U2.3 (VO), U4.14 (VCC), U4.14 (VCC), U4.14 (VCC), U4.14 (VCC), U4.14 (VCC)
- net V_ENV_BIAS: now also R22.2, R23.2, R6.2
- new net: C21.1, Q5.1 (B), Q5.2 (E), R20.2, RV3.2, RV3.3, U5.1
- new net: C21.2, R18.1, RV3.1, U5.2 (-)
- new net: C19.1, L3.2, U5.3 (+)
- new net: C23.1, C25.2, Q5.3 (C), R22.1, U3.10 (+)
- new net: C25.1, R24.2
- new net: Q7.1 (B), R24.1, R26.2, R27.1
- new net: Q7.3 (C), R26.1, R30.2, R32.2
- new net: R32.1, U4.5
- new net: J11.1 (P1), U4.6
- new net: J7.1 (P1), R20.1
- new net: J9.1 (P1), U3.8, U3.9 (-)
- new net: C4.1, L2.2, U1.5 (+)
- new net: C8.2, R2.1, RV2.1, U1.6 (-)
- new net: C8.1, Q2.1 (B), Q2.2 (E), R4.2, RV2.2, RV2.3, U1.7
- new net: C14.1, C16.2, Q2.3 (C), R6.1, U3.5 (+)
- new net: C16.1, R9.2
- new net: Q4.1 (B), R12.2, R13.1, R9.1
- new net: Q4.3 (C), R12.1, R15.2, R17.2
- new net: R17.1, U4.3
- new net: J6.1 (P1), U4.4
- new net: J2.1 (P1), R4.1
- new net: J4.1 (P1), U3.6 (-), U3.7
- new net: C20.1, L4.2, U5.5 (+)
- new net: C22.2, R19.1, RV4.1, U5.6 (-)
- new net: C22.1, Q6.1 (B), Q6.2 (E), R21.2, RV4.2, RV4.3, U5.7
- new net: C24.1, C26.2, Q6.3 (C), R23.1, U3.12 (+)
- new net: C26.1, R25.2
- new net: Q8.1 (B), R25.1, R28.2, R29.1
- new net: Q8.3 (C), R28.1, R31.2, R33.2
- new net: R33.1, U4.9
- new net: J12.1 (P1), U4.8
- new net: J8.1 (P1), R21.1
- new net: J10.1 (P1), U3.13 (-), U3.14
Other:
- note added: "+5V"
- moved on the sheet: C11, J5, U4A

Commit message: ^XPhone Input Board layout; +bug record
Parts:
- U2: symbol 78L05 -> 78L05-RESCUE-Input_Board
Connections:
- net +12V: now also U2.3 (VI); no longer U2.1 (VI)
- net VCC: now also U2.1 (VO); no longer U2.3 (VO)
Changed lines of the file:
@@
 EESchema Schematic File Version 2
+LIBS:Input Board-rescue
 LIBS:device
 LIBS:transistors
@@
 $EndComp
 $Comp
-L 78L05 U2
+L 78L05-RESCUE-Input_Board U2
 U 1 1 59620FB2
 P 2650 6450
