File: Analog Synth/ScreamFilter/ScreamFilter.brd (EAGLE design)
At the start: 46.4 x 63.5 mm, 37 parts, among them IC1 TL084P, IC2 TL082P, Q1 J310, Q2 J310, Q3 J310, Q4 J310

Commit message: working on ScreamFilter DIY layout
Parts:
- moved R16 28.8 mm to (37.5, 25.4), turned to 270 degrees
- moved R15 28.6 mm to (37.5, 43.2), turned to 90 degrees
- moved C5 24.2 mm to (35.6, 55.9)
- moved C6 24.2 mm to (35.6, 12.7)
- moved C7 24.2 mm to (35.6, 50.8)
- moved C8 24.2 mm to (35.6, 17.8)
- moved U$1 22.9 mm to (31.8, 34.3)
- moved FEEDBACK 16.6 mm to (21.0, 40.0)
- moved C4 16.6 mm to (11.4, 4.45)
- moved IC1 16.6 mm to (16.5, 17.8)
- moved Q4 16.6 mm to (16.5, 6.35)
- moved R18 16.6 mm to (2.54, 47.6)
- moved R2 16.6 mm to (19.1, 55.2)
- moved R3 16.6 mm to (19.1, 53.3)
- moved R4 16.6 mm to (19.7, 47.6)
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Routing:
- net GND: track 148.0 -> 204.0 mm, vias 0 -> 2
- net -12V: track 38.8 -> 73.3 mm, vias 0 -> 4
- net N$10: track 18.2 -> 51.0 mm, vias 0 -> 1
- net +12V: track 53.8 -> 69.5 mm, vias 0 -> 2
- net N$1: track 4.07 -> 4.60 mm
- added copper zone on layer 16, net GND
Other:
- board size 46.4 x 63.5 mm -> 38.7 x 62.2 mm
- board text added: "Jensen"
- board text added: "Ryan"
- board text added: "Scream Filter"

Commit message: PS-VCO, ScreamFilter, VCA-v2, and XPhone stuff. (something I must have done 2 years ago...)
Parts:
- R4: value 1k -> 100
Changed lines of the file:
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@@
 <grid distance="0.05" unitdist="inch" unit="inch" style="lines" multiple="1" display="no" altdistance="0.025" altunitdist="inch" altunit="inch"/>
 <layers>
-<layer number="1" name="Top" color="4" fill="1" visible="no" active="yes"/>
+<layer number="1" name="Top" color="4" fill="1" visible="yes" active="yes"/>
 <layer number="2" name="Route2" color="1" fill="3" visible="no" active="no"/>
 <layer number="3" name="Route3" color="4" fill="3" visible="no" active="no"/>
@@
 <layer number="18" name="Vias" color="2" fill="1" visible="yes" active="yes"/>
 <layer number="19" name="Unrouted" color="6" fill="1" visible="yes" active="yes"/>
-<layer number="20" name="Dimension" color="15" fill="1" visible="no" active="yes"/>
-<layer number="21" name="tPlace" color="7" fill="1" visible="no" active="yes"/>
-<layer number="22" name="bPlace" color="7" fill="1" visible="no" active="yes"/>
-<layer number="23" name="tOrigins" color="15" fill="1" visible="no" active="yes"/>
-<layer number="24" name="bOrigins" color="15" fill="1" visible="no" active="yes"/>
-<layer number="25" name="tNames" color="7" fill="1" visible="no" active="yes"/>
-<layer number="26" name="bNames" color="7" fill="1" visible="no" active="yes"/>
-<layer number="27" name="tValues" color="7" fill="1" visible="no" active="yes"/>
-<layer number="28" name="bValues" color="7" fill="1" visible="no" active="yes"/>
+<layer number="20" name="Dimension" color="15" fill="1" visible="yes" active="yes"/>
+<layer number="21" name="tPlace" color="7" fill="1" visible="yes" active="yes"/>
+<layer number="22" name="bPlace" color="7" fill="1" visible="yes" active="yes"/>
+<layer number="23" name="tOrigins" color="15" fill="1" visible="yes" active="yes"/>
+<layer number="24" name="bOrigins" color="15" fill="1" visible="yes" active="yes"/>
+<layer number="25" name="tNames" color="7" fill="1" visible="yes" active="yes"/>
+<layer number="26" name="bNames" color="7" fill="1" visible="yes" active="yes"/>
+<layer number="27" name="tValues" color="7" fill="1" visible="yes" active="yes"/>
+<layer number="28" name="bValues" color="7" fill="1" visible="yes" active="yes"/>
 <layer number="29" name="tStop" color="7" fill="3" visible="no" active="yes"/>
 <layer number="30" name="bStop" color="7" fill="6" visible="no" active="yes"/>
@@
 <element name="R2" library="rcl" package="0204/7" value="100k" x="19.05" y="55.245" rot="R180"/>
 <element name="R3" library="rcl" package="0204/7" value="100" x="19.05" y="53.34" rot="R180"/>
-<element name="R4" library="rcl" package="0204/7" value="1k" x="19.685" y="47.625" rot="R90"/>
+<element name="R4" library="rcl" package="0204/7" value="100" x="19.685" y="47.625" rot="R90"/>
 <element name="Q2" library="transistor-small-signal" package="TO92R" value="J310" x="7.62" y="27.305" rot="R180"/>
 <element name="C2" library="rcl" package="C025-025X050" value="2.2n" x="7.62" y="21.59" rot="R270"/>
@@
 <wire x1="3.81" y1="8.255" x2="7.62" y2="4.445" width="0.4064" layer="16"/>
 <wire x1="7.62" y1="4.445" x2="10.16" y2="4.445" width="0.4064" layer="16"/>
-<polygon width="0.4064" layer="16" isolate="1.016">
+<polygon width="0.4064" layer="16" isolate="1.016" orphans="yes">
 <vertex x="0" y="62.23"/>
 <vertex x="0" y="0"/>
